File: OpenDropV2/DesignFiles/OpenDropV2.sch (KiCad schematic (older format))
At the start: 225 parts, among them J1 DC_JACK, P1 CONN_01X01, P10 CONN_01X01, P11 CONN_01X01, P12 CONN_01X01, P13 ScrewPad1, P14 ScrewPad2, P15 ScrewPad3, P16 ScrewPad4, P2 CONN_01X01, P3 CONN_01X01, P5 CONN_01X01, P6 CONN_01X30, P7 CONN_01X01, P8 CONN_01X01, P9 CONN_01X01, Q1 BSS138, Q2 BSS138, Q3 BSS138, Q5 BSS138, Q6 BSS138, Q7 BSS138, SW1 SW_PUSH, SW2 SW_PUSH, SW5 SPST, T1 IRF 840S, U1 MAX1771ESA, U2 HV507, U3 ARDUINO_MICRO, U4 HV507, U5 ESP8266_SMD, U6 MCP6002

Commit message: Random changes just from firing up the project
adjusted libraries to match my paths
Parts:
- Q1, Q2, Q3, Q5, Q6, Q7: symbol BSS138 -> BSS138-RESCUE-OpenDropV2
Changed lines of the file:
@@
 LIBS:contrib
 LIBS:valves
+LIBS:ESP8266
 LIBS:GaudiLabsPartsLibrary
 LIBS:OpenDropV2-cache
-EELAYER 26 0
+EELAYER 25 0
 EELAYER END
 $Descr A3 16535 11693
@@
 3.3V
 $Comp
-L BSS138 Q2
+L BSS138-RESCUE-OpenDropV2 Q2
 U 1 1 565B696F
 P 12300 7500
@@
 $EndComp
 $Comp
-L BSS138 Q1
+L BSS138-RESCUE-OpenDropV2 Q1
 U 1 1 565B91C1
 P 11850 7400
@@
 LED_LIGHT
 $Comp
-L BSS138 Q3
+L BSS138-RESCUE-OpenDropV2 Q3
 U 1 1 565AB267
 P 9950 9450
@@
 3.3V
 $Comp
-L BSS138 Q5
+L BSS138-RESCUE-OpenDropV2 Q5
 U 1 1 5732C8D0
 P 7450 8750
@@
 ESP_GPIO0
 $Comp
-L BSS138 Q6
+L BSS138-RESCUE-OpenDropV2 Q6
 U 1 1 5733DD94
 P 10550 8700
@@
 $EndComp
 $Comp
-L BSS138 Q7
+L BSS138-RESCUE-OpenDropV2 Q7
 U 1 1 5733E045
 P 10850 8350
